Commit message: low level planner finished

File: ur16e_dual_arm_description/urdf/dual_arm.xacro (robot description, xacro)
@@ -12,10 +12,10 @@
     <parent link="world" />
     <child link = "left_base_link" />
-    <origin xyz="-0.5 0 0" rpy="0 0 0" />
+    <origin xyz="-0.351 0.535 -0.012" rpy="-0.003 -0.015 2.788" />
   </joint>
   <joint name="world_to_right" type="fixed">
     <parent link="world" />
     <child link = "right_base_link" />
-    <origin xyz="0.5 0 0" rpy="0 0 0" />
+    <origin xyz="0.557 0.520 -0.005" rpy="-0.037 0.005 -2.838" />
   </joint>
 </robot>

Commit message: arm calibration done

File: ur16e_dual_arm_description/urdf/dual_arm.xacro (robot description, xacro)
@@ -12,10 +12,10 @@
     <parent link="world" />
     <child link = "left_base_link" />
-    <origin xyz="-0.351 0.535 -0.012" rpy="-0.003 -0.015 2.788" />
+    <origin xyz="0.342 0.654 0.007" rpy="-0.006 -0.008 1.573" />
   </joint>
   <joint name="world_to_right" type="fixed">
     <parent link="world" />
     <child link = "right_base_link" />
-    <origin xyz="0.557 0.520 -0.005" rpy="-0.037 0.005 -2.838" />
+    <origin xyz="0.368 -0.500 -.025" rpy="-0.019 -0.047 1.582" />
   </joint>
 </robot>
