Commit message: added benchmarking script for calibration

File: ur16e_dual_arm_description/urdf/dual_arm_left_calibrator.urdf (robot description, URDF)
Before this commit: robot dual_arm_ur16e, 27 links, 26 joints
Links:
- link left_suction_gripper: geometry collision cylinder length=0.15 radius=0.05; visual mesh filename=package://ur16e_dual_arm_description/urdf/meshes/calibrator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 scale=0.001 0.001 0.001
Joints:
- joint left_wrist_3_link-suction_gripper: origin xyz=0 0 0.0 rpy=0 0 3.14 -> xyz=0 0 0.0 rpy=0 0 0

Commit message: critical stuff done

File: ur16e_dual_arm_description/urdf/dual_arm_left_calibrator.urdf (robot description, URDF)
Before this commit: robot dual_arm_ur16e, 27 links, 26 joints
Joints:
- joint left_suction_gripper-poi: origin xyz=-0.003 -0.001 0.093 rpy=0 0 0 -> xyz=-0.003 -0.001 0.083 rpy=0 0 0
