Commit message: added rws_gripper urdf and mesh, WIP

File: ur16e_dual_arm_description/urdf/dual_arm_left_suction_gripper_right_rws_gripper.urdf (robot description, URDF)
Before this commit: robot dual_arm_ur16e, 27 links, 26 joints
Links:
- link right_suction_gripper: geometry collision cylinder length=0.22 radius=0.05; visual mesh filename=package://ur16e_dual_arm_description/urdf/meshes/rws.STL scale=0.001 0.001 0.001
Joints:
- joint world_to_left: origin xyz=-0.363 0.521 0.008 rpy=-0.003 -0.017 1.583 -> xyz=-0.498 0.530 0.005 rpy=-0.008 0.002 2.237
- joint world_to_right: origin xyz=0.576 0.525 0.007 rpy=0.004 -0.033 -1.590 -> xyz=0.647 0.539 0.007 rpy=-0.002 -0.001 2.268
