Commit message: stable

File: ur16e_dual_arm_description/urdf/dual_arm.urdf (robot description, URDF)
Before this commit: robot dual_arm_ur16e, 23 links, 22 joints
Links:
- added link left_suction_gripper, mass 0.1; collision cylinder length=0.22 radius=0.05; visual cylinder length=0.22 radius=0.05
- added link left_suction_gripper_poi
- added link right_suction_gripper, mass 0.1; collision cylinder length=0.22 radius=0.05; visual cylinder length=0.22 radius=0.05
- added link right_suction_gripper_poi
Joints:
- added joint left_suction_gripper-poi: type fixed, parent left_suction_gripper, child left_suction_gripper_poi, origin xyz=0 0 0.11 rpy=0 0 0
- added joint left_wrist_3_link-suction_gripper: type fixed, parent left_wrist_3_link, child left_suction_gripper, origin xyz=0 0 0.11 rpy=0 0 0
- added joint right_suction_gripper-poi: type fixed, parent right_suction_gripper, child right_suction_gripper_poi, origin xyz=0 0 0.11 rpy=0 0 0
- added joint right_wrist_3_link-_suction_gripper: type fixed, parent right_wrist_3_link, child right_suction_gripper, origin xyz=0 0 0.11 rpy=0 0 0
- joint world_to_left: origin xyz=-0.5 0 0 rpy=0 0 0 -> xyz=-0.510 0.565 0.013 rpy=-0.013 -0.015 2.259
- joint world_to_right: origin xyz=0.5 0 0 rpy=0 0 0 -> xyz=0.636 0.617 0.005 rpy=-0.007 -0.032 2.295

File: ur16e_dual_arm_description/urdf/dual_arm.xacro (robot description, xacro)
@@ -12,10 +12,10 @@
     <parent link="world" />
     <child link = "left_base_link" />
-    <origin xyz="0.342 0.654 0.007" rpy="-0.006 -0.008 1.573" />
+    <origin xyz="-0.660 0.554 0.010" rpy="-0.006 -0.008 1.573" />
   </joint>
   <joint name="world_to_right" type="fixed">
     <parent link="world" />
     <child link = "right_base_link" />
-    <origin xyz="0.368 -0.500 -.025" rpy="-0.019 -0.047 1.582" />
+    <origin xyz="0.660 0.554 0.010" rpy="-0.007 0.023 2.163" />
   </joint>
 </robot>

Commit message: latest commit

File: ur16e_dual_arm_description/urdf/dual_arm.urdf (robot description, URDF)
Before this commit: robot dual_arm_ur16e, 27 links, 26 joints
Links:
- link left_suction_gripper: geometry collision cylinder length=0.15 radius=0.05; visual mesh filename=package://ur16e_dual_arm_description/urdf/meshes/suction_gr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 scale=0.001 0.001 0.001
Joints:
- joint left_suction_gripper-poi: origin xyz=0 0 0.19 rpy=0 0 0 -> xyz=-0.004 -0.002 0.173 rpy=0 0 0
- joint world_to_left: origin xyz=-0.510 0.565 0.013 rpy=-0.013 -0.015 2.259 -> xyz=-0.498 0.530 0.005 rpy=-0.008 0.002 2.237
- joint world_to_right: origin xyz=0.636 0.617 0.005 rpy=-0.007 -0.032 2.295 -> xyz=0.647 0.539 0.007 rpy=-0.002 -0.001 2.268

Commit message: camera launch added and calibrator ee calibrated

File: ur16e_dual_arm_description/urdf/dual_arm.urdf (robot description, URDF)
Before this commit: robot dual_arm_ur16e, 27 links, 26 joints
Links:
- link left_suction_gripper: geometry collision cylinder length=0.15 radius=0.05; visual mesh filename=package://ur16e_dual_arm_description/urdf/meshes/calibrator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 scale=0.001 0.001 0.001
Joints:
- joint left_suction_gripper-poi: origin xyz=-0.004 -0.002 0.173 rpy=0 0 0 -> xyz=-0.003 -0.001 0.093 rpy=0 0 0
- joint left_wrist_3_link-suction_gripper: origin xyz=0 0 0.0 rpy=0 0 3.14 -> xyz=0 0 0.0 rpy=0 0 0

File: ur16e_dual_arm_description/urdf/dual_arm_left_calibrator.urdf (robot description, URDF)
Before this commit: robot dual_arm_ur16e, 27 links, 26 joints
Joints:
- joint left_suction_gripper-poi: origin xyz=-0.004 -0.002 0.173 rpy=0 0 0 -> xyz=-0.003 -0.001 0.093 rpy=0 0 0

Commit message: cameras integrated with new system

File: ur16e_dual_arm_description/urdf/dual_arm.urdf (robot description, URDF)
Before this commit: robot dual_arm_ur16e, 27 links, 26 joints
Joints:
- joint world_to_left: origin xyz=-0.498 0.530 0.005 rpy=-0.008 0.002 2.237 -> xyz=-0.3906717303685856 0.4086080874800634 0.009765414138713466 rpy=0.0030070500195190893 -0.0073779695804560555 1.561587737833231

Commit message: setup second table, debugging perception

File: ur16e_dual_arm_description/urdf/dual_arm.urdf (robot description, URDF)
Before this commit: robot dual_arm_ur16e, 27 links, 26 joints
Links:
- link left_suction_gripper: geometry collision cylinder length=0.15 radius=0.05; visual mesh filename=package://ur16e_dual_arm_description/urdf/meshes/suction_gr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 scale=0.001 0.001 0.001
Joints:
- joint left_suction_gripper-poi: origin xyz=-0.003 -0.001 0.093 rpy=0 0 0 -> xyz=-0.004 -0.002 0.173 rpy=0 0 0
- joint left_wrist_3_link-suction_gripper: origin xyz=0 0 0.0 rpy=0 0 0 -> xyz=0 0 0.0 rpy=0 0 3.14
- joint world_to_left: origin xyz=-0.3906717303685856 0.4086080874800634 0.009765414138713466 rpy=0.0030070500195190893 -0.0073779695804560555 1.561587737833231 -> xyz=-0.363 0.521 0.008 rpy=-0.003 -0.017 1.583
- joint world_to_right: origin xyz=0.647 0.539 0.007 rpy=-0.002 -0.001 2.268 -> xyz=0.576 0.525 0.007 rpy=0.004 -0.033 -1.590

Commit message: updated urdf to add rws gripper and calibrated rws ee

File: ur16e_dual_arm_description/urdf/dual_arm.urdf (robot description, URDF)
Before this commit: robot dual_arm_ur16e, 27 links, 26 joints
Links:
- link right_suction_gripper: geometry collision cylinder length=0.22 radius=0.05; visual mesh filename=package://ur16e_dual_arm_description/urdf/meshes/rws.STL scale=0.001 0.001 0.001
Joints:
- joint right_suction_gripper-poi: origin xyz=0 0 0.11 rpy=0 0 0 -> xyz=-0.005 -0.004 0.109 rpy=0 0 0
- joint right_wrist_3_link-_suction_gripper: origin xyz=0 0 0.11 rpy=0 0 0 -> xyz=0 0 0 rpy=0 0 0
- joint world_to_left: origin xyz=-0.363 0.521 0.008 rpy=-0.003 -0.017 1.583 -> xyz=-0.498 0.530 0.005 rpy=-0.008 0.002 2.237
- joint world_to_right: origin xyz=0.576 0.525 0.007 rpy=0.004 -0.033 -1.590 -> xyz=0.647 0.539 0.007 rpy=-0.002 -0.001 2.268

File: ur16e_dual_arm_description/urdf/dual_arm_left_suction_gripper_right_rws_gripper.urdf (robot description, URDF)
Before this commit: robot dual_arm_ur16e, 27 links, 26 joints
Joints:
- joint right_suction_gripper-poi: origin xyz=0 0 0.11 rpy=0 0 0 -> xyz=-0.005 -0.004 0.109 rpy=0 0 0
- joint right_wrist_3_link-_suction_gripper: origin xyz=0 0 0.11 rpy=0 0 0 -> xyz=0 0 0 rpy=0 0 0

Commit message: world calibration error after last commit, applied fix

File: ur16e_dual_arm_description/urdf/dual_arm.urdf (robot description, URDF)
Before this commit: robot dual_arm_ur16e, 27 links, 26 joints
Joints:
- joint world_to_left: origin xyz=-0.498 0.530 0.005 rpy=-0.008 0.002 2.237 -> xyz=-0.363 0.521 0.008 rpy=-0.003 -0.017 1.583

Commit message: solved the world calibration issue, allss goooood

File: ur16e_dual_arm_description/urdf/dual_arm.urdf (robot description, URDF)
Before this commit: robot dual_arm_ur16e, 27 links, 26 joints
Joints:
- joint world_to_right: origin xyz=0.647 0.539 0.007 rpy=-0.002 -0.001 2.268 -> xyz=0.576 0.525 0.007 rpy=0.004 -0.033 -1.590
